File: drawing tablet analog frontend.kicad_pcb (KiCad board)
At the start: 2 copper layers, 22.5 x 13 mm, 41 parts, among them J1 Conn_01x09, Q1 AO3400A, Q2 AO3400A, Q3 AO3400A, U1 COS8054TR

Commit message: Add 1n capacitor on inhibit, ~1us delay
Parts:
- added C4: 1n, Capacitor_SMD:C_0402_1005Metric, F.Cu at (53.8, 43.4)
- renumbered C9 to C10, C10 to C11, C11 to C12, C12 to C13, C13 to C14, C14 to C15, C15 to C16, C16 to C17, C17 to C18, C4 to C5, C5 to C6, C6 to C7, C7 to C8, C8 to C9
Routing:
- net Net-(Q1-G): track 1.64 -> 2.41 mm
- net GND: track 28.4 -> 29.1 mm, vias 35 -> 34
